Commit message: Add: ackermann car

File: linorobot2_description/urdf/mech/base.urdf.xacro (robot description, xacro)
@@ -1,9 +1,9 @@
 <?xml version="1.0"?>
 <robot xmlns:xacro="http://ros.org/wiki/xacro">
-  <xacro:macro name="base" params="length width height mass wheel_radius wheel_pos_z">
+  <xacro:macro name="base" params="x y z length width height mass wheel_radius wheel_pos_z">
     <link name="base_footprint"/>
     <link name="base_link">
       <visual>
-        <origin xyz="0 0 0" rpy="0 0 0"/>
+        <origin xyz="${x} ${y} ${z}" rpy="0 0 0"/>
         <geometry>
           <box size="${length} ${width} ${height}"/>
